File: Demoproject/BMS/BMS.kicad_pcb (KiCad board)
At the start: 2 copper layers, 34 x 32 mm, 33 parts, among them IC1 HY2213-BB3A, IC2 HY2213-BB3A, IC3 HY2213-BB3A, IC4 HY2213-BB3A, IC5 HY2213-BB3A, IC6 HY2213-BB3A, IC7 HY2213-BB3A, IC8 HY2213-BB3A, J1 Conn_02x09_Odd_Even, Q1 AO3400A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

Commit message: powerpoint update
Parts:
- added R10: 75R, Resistor_SMD:R_0805_2012Metric, F.Cu at (105.1, 65.0)
- added R11: 75R, Resistor_SMD:R_0805_2012Metric, F.Cu at (112.0, 65.0)
- added R12: 75R, Resistor_SMD:R_0805_2012Metric, F.Cu at (94.9, 98.0)
- added R13: 75R, Resistor_SMD:R_0805_2012Metric, F.Cu at (100.0, 98.0)
- added R14: 75R, Resistor_SMD:R_0805_2012Metric, F.Cu at (106.9, 98.0)
- added R15: 75R, Resistor_SMD:R_0805_2012Metric, F.Cu at (113.0, 98.0)
- added R16: 75R, Resistor_SMD:R_0805_2012Metric, F.Cu at (119.1, 98.0)
- added R9: 75R, Resistor_SMD:R_0805_2012Metric, F.Cu at (99.9, 65.0)
Connections:
- Q1 pad 3: B0 -> Net-(Q1-Pad3)
- Q2 pad 3: B1 -> Net-(Q2-Pad3)
- Q3 pad 3: B2 -> Net-(Q3-Pad3)
- Q4 pad 3: B3 -> Net-(Q4-Pad3)
- Q5 pad 3: B4 -> Net-(Q5-Pad3)
- Q6 pad 3: B5 -> Net-(Q6-Pad3)
- Q7 pad 3: B6 -> Net-(Q7-Pad3)
- Q8 pad 3: B7 -> Net-(Q8-Pad3)
Routing:
- net Net-(C2-Pad1): track 1.80 -> 9.02 mm, vias 0 -> 2
- net Net-(Q6-Pad3): track 0.00 -> 7.02 mm, vias 0 -> 2
- net Net-(Q7-Pad3): track 0.00 -> 6.97 mm, vias 0 -> 2
- net Net-(Q5-Pad3): track 0.00 -> 6.80 mm, vias 0 -> 2
- net Net-(Q4-Pad3): track 0.00 -> 5.80 mm, vias 0 -> 2
- net Net-(Q3-Pad3): track 0.00 -> 5.50 mm, vias 0 -> 2
- net GND: track 9.39 -> 14.6 mm, vias 2 -> 4
- net B4: track 53.6 -> 57.8 mm
- net Net-(Q1-Pad3): track 0.00 -> 3.97 mm
- net Net-(Q8-Pad3): track 0.00 -> 3.90 mm
- net Net-(Q2-Pad3): track 0.00 -> 3.55 mm
- net B3: track 50.1 -> 52.4 mm, vias 2 -> 3
- net B2: track 24.5 -> 22.6 mm
- net B5: track 24.6 -> 23.0 mm
- net B6: track 23.6 -> 22.0 mm
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Other:
- board size 34 x 32 mm -> 34 x 37 mm
