File: Demoproject/BMS/bmsCell.kicad_sch (KiCad schematic)
At the start: 4 parts, among them IC3 HY2213-BB3A, Q3 AO3400A

Commit message: powerpoint update
Parts:
- added R?: 75R, Resistor_SMD:R_0805_2012Metric, symbol Device:R_Small
- renumbered C3 to C1, IC3 to IC1, Q3 to Q1, R3 to R1
Connections:
- net BA: now also R?.1; no longer Q1.3 (D)
- new net: Q1.3 (D), R?.2
Changed lines of the file:
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@@
 (kicad_sch (version 20211123) (generator eeschema)
   (paper "A4")
+  (junction (at 77.47 46.99) (diameter 0) (color 0 0 0 0)
+  )
   (junction (at 77.47 63.5) (diameter 0) (color 0 0 0 0)
-  )
-  (junction (at 77.47 46.99) (diameter 0) (color 0 0 0 0)
   )
   (wire (pts (xy 73.66 46.99) (xy 77.47 46.99))
@@
     (stroke (width 0) (type default) (color 0 0 0 0))
   )
-  (wire (pts (xy 77.47 53.34) (xy 77.47 46.99))
+  (wire (pts (xy 77.47 46.99) (xy 105.41 46.99))
     (stroke (width 0) (type default) (color 0 0 0 0))
   )
@@
     (stroke (width 0) (type default) (color 0 0 0 0))
   )
-  (wire (pts (xy 77.47 46.99) (xy 105.41 46.99))
+  (wire (pts (xy 77.47 46.99) (xy 77.47 48.26))
     (stroke (width 0) (type default) (color 0 0 0 0))
   )
@@
   (symbol (lib_id "Device:C_Small") (at 109.22 58.42 0)
     (in_bom yes) (on_board yes) (fields_autoplaced)
-    (property "Reference" "C3" (id 0) (at 111.5441 57.5178 0)
+    (property "Reference" "C1" (id 0) (at 111.5441 57.5178 0)
       (effects (font (size 1.27 1.27)) (justify left))
     )
@@
   (symbol (lib_id "Transistor_FET:AO3400A") (at 80.01 58.42 0) (mirror y)
     (in_bom yes) (on_board yes) (fields_autoplaced)
-    (property "Reference" "Q3" (id 0) (at 74.8031 57.5115 0)
+    (property "Reference" "Q1" (id 0) (at 74.8031 57.5115 0)
       (effects (font (size 1.27 1.27)) (justify left))
     )
@@
   (symbol (lib_id "Device:R_Small") (at 105.41 49.53 0)
     (in_bom yes) (on_board yes) (fields_autoplaced)
-    (property "Reference" "R3" (id 0) (at 106.9086 48.6215 0)
+    (property "Reference" "R1" (id 0) (at 106.9086 48.6215 0)
       (effects (font (size 1.27 1.27)) (justify left))
     )
@@
     (pin "2")
   )
+  (symbol (lib_id "Device:R_Small") (at 77.47 50.8 0)
+    (in_bom yes) (on_board yes) (fields_autoplaced)
+    (property "Reference" "R?" (id 0) (at 78.9686 49.8915 0)
+      (effects (font (size 1.27 1.27)) (justify left))
+    )
+    (property "Value" "75R" (id 1) (at 78.9686 52.6666 0)
+      (effects (font (size 1.27 1.27)) (justify left))
+    )
+    (property "Footprint" "Resistor_SMD:R_0805_2012Metric" (id 2) (at 77.47 50.8 0)
+      (effects (font (size 1.27 1.27)) hide)
+    )
+    (property "Datasheet" "~" (id 3) (at 77.47 50.8 0)
+      (effects (font (size 1.27 1.27)) hide)
+    )
+    (pin "1")
+    (pin "2")
+  )
   (symbol (lib_id "SamacSys_Parts:HY2213-BB3A") (at 107.95 60.96 180)
     (in_bom yes) (on_board yes) (fields_autoplaced)
-    (property "Reference" "IC3" (id 0) (at 95.25 49.5005 0))
+    (property "Reference" "IC1" (id 0) (at 95.25 49.5005 0))
     (property "Value" "HY2213-BB3A" (id 1) (at 95.25 52.2756 0))
     (property "Footprint" "SamacSys_Parts:SOT95P280X140-6N" (id 2) (at 83.82 63.5 0)

Commit message: update
Parts:
- gave numbers to parts that had none: 1
- renumbered C1 to C8, IC1 to IC8, Q1 to Q8, R1 to R8
Changed lines of the file:
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@@
   (symbol (lib_id "Device:C_Small") (at 109.22 58.42 0)
     (in_bom yes) (on_board yes) (fields_autoplaced)
-    (property "Reference" "C1" (id 0) (at 111.5441 57.5178 0)
+    (property "Reference" "C8" (id 0) (at 111.5441 57.5178 0)
       (effects (font (size 1.27 1.27)) (justify left))
     )
@@
   (symbol (lib_id "Transistor_FET:AO3400A") (at 80.01 58.42 0) (mirror y)
     (in_bom yes) (on_board yes) (fields_autoplaced)
-    (property "Reference" "Q1" (id 0) (at 74.8031 57.5115 0)
+    (property "Reference" "Q8" (id 0) (at 74.8031 57.5115 0)
       (effects (font (size 1.27 1.27)) (justify left))
     )
@@
   (symbol (lib_id "Device:R_Small") (at 105.41 49.53 0)
     (in_bom yes) (on_board yes) (fields_autoplaced)
-    (property "Reference" "R1" (id 0) (at 106.9086 48.6215 0)
+    (property "Reference" "R8" (id 0) (at 106.9086 48.6215 0)
       (effects (font (size 1.27 1.27)) (justify left))
     )
@@
   (symbol (lib_id "Device:R_Small") (at 77.47 50.8 0)
     (in_bom yes) (on_board yes) (fields_autoplaced)
-    (property "Reference" "R?" (id 0) (at 78.9686 49.8915 0)
+    (property "Reference" "R16" (id 0) (at 78.9686 49.8915 0)
       (effects (font (size 1.27 1.27)) (justify left))
     )
@@
   (symbol (lib_id "SamacSys_Parts:HY2213-BB3A") (at 107.95 60.96 180)
     (in_bom yes) (on_board yes) (fields_autoplaced)
-    (property "Reference" "IC1" (id 0) (at 95.25 49.5005 0))
+    (property "Reference" "IC8" (id 0) (at 95.25 49.5005 0))
     (property "Value" "HY2213-BB3A" (id 1) (at 95.25 52.2756 0))
     (property "Footprint" "SamacSys_Parts:SOT95P280X140-6N" (id 2) (at 83.82 63.5 0)
