File: Demoproject/USBMIc/USBMIc.kicad_sch (KiCad schematic)
At the start: 33 parts, among them J1 USB_B_Micro, J2 Prog, SW1 SW_Push, SW2 SW_Push, U1 USBLC6-2SC6, U2 LP5907MFX-3.3, U3 STM32F446RCTx, X1 ACO-xxxMHz, Y1 SG-8018CB_12.2880M-TJHPA3

Commit message: pcb layout
Parts:
- gave numbers to parts that had none: 6
Changed lines of the file:
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@@
   (symbol (lib_id "Device:C_Small") (at 152.4 29.21 0) (unit 1)
     (in_bom yes) (on_board yes) (fields_autoplaced)
-    (property "Reference" "C?" (id 0) (at 154.7241 28.3078 0)
+    (property "Reference" "C11" (id 0) (at 154.7241 28.3078 0)
       (effects (font (size 1.27 1.27)) (justify left))
     )
@@
   (symbol (lib_id "Device:C_Small") (at 137.16 29.21 0) (unit 1)
     (in_bom yes) (on_board yes) (fields_autoplaced)
-    (property "Reference" "C?" (id 0) (at 139.4841 28.3078 0)
+    (property "Reference" "C9" (id 0) (at 139.4841 28.3078 0)
       (effects (font (size 1.27 1.27)) (justify left))
     )
@@
   (symbol (lib_id "Device:C_Small") (at 160.02 29.21 0) (unit 1)
     (in_bom yes) (on_board yes) (fields_autoplaced)
-    (property "Reference" "C?" (id 0) (at 162.3441 28.3078 0)
+    (property "Reference" "C12" (id 0) (at 162.3441 28.3078 0)
       (effects (font (size 1.27 1.27)) (justify left))
     )
@@
   (symbol (lib_id "Device:C_Small") (at 144.78 29.21 0) (unit 1)
     (in_bom yes) (on_board yes) (fields_autoplaced)
-    (property "Reference" "C?" (id 0) (at 147.1041 28.3078 0)
+    (property "Reference" "C10" (id 0) (at 147.1041 28.3078 0)
       (effects (font (size 1.27 1.27)) (justify left))
     )
@@
   (symbol (lib_id "Device:C_Small") (at 167.64 29.21 0) (unit 1)
     (in_bom yes) (on_board yes) (fields_autoplaced)
-    (property "Reference" "C?" (id 0) (at 169.9641 28.3078 0)
+    (property "Reference" "C13" (id 0) (at 169.9641 28.3078 0)
       (effects (font (size 1.27 1.27)) (justify left))
     )
@@
   (symbol (lib_id "Device:C_Small") (at 175.26 29.21 0) (unit 1)
     (in_bom yes) (on_board yes)
-    (property "Reference" "C?" (id 0) (at 180.34 27.94 0)
+    (property "Reference" "C14" (id 0) (at 180.34 27.94 0)
       (effects (font (size 1.27 1.27)) (justify left))
     )
@@
       (reference "C8") (unit 1) (value "100nF") (footprint "Capacitor_SMD:C_0603_1608Metric")
     )
+    (path "/8674a9ad-d287-480a-9b7e-298ec5791677"
+      (reference "C9") (unit 1) (value "1uF") (footprint "Capacitor_SMD:C_0603_1608Metric")
+    )
+    (path "/acb5489d-7f48-415d-95ac-a67b3110aa0e"
+      (reference "C10") (unit 1) (value "1uF") (footprint "Capacitor_SMD:C_0603_1608Metric")
+    )
     (path "/0e9f942e-04a2-4967-a20f-0322f433a2b7"
-      (reference "C?") (unit 1) (value "1uF") (footprint "Capacitor_SMD:C_0603_1608Metric")
-    )
-    (path "/8674a9ad-d287-480a-9b7e-298ec5791677"
-      (reference "C?") (unit 1) (value "1uF") (footprint "Capacitor_SMD:C_0603_1608Metric")
+      (reference "C11") (unit 1) (value "1uF") (footprint "Capacitor_SMD:C_0603_1608Metric")
     )
     (path "/a0c16cd7-a3f1-46d5-8625-1006ed98f1d6"
-      (reference "C?") (unit 1) (value "1uF") (footprint "Capacitor_SMD:C_0603_1608Metric")
-    )
-    (path "/acb5489d-7f48-415d-95ac-a67b3110aa0e"
-      (reference "C?") (unit 1) (value "1uF") (footprint "Capacitor_SMD:C_0603_1608Metric")
+      (reference "C12") (unit 1) (value "1uF") (footprint "Capacitor_SMD:C_0603_1608Metric")
     )
     (path "/b17def37-70d0-4433-8253-4a61b7eecee8"
-      (reference "C?") (unit 1) (value "1uF") (footprint "Capacitor_SMD:C_0603_1608Metric")
+      (reference "C13") (unit 1) (value "1uF") (footprint "Capacitor_SMD:C_0603_1608Metric")
     )
     (path "/ee219667-dd08-4087-878d-660b5160b21f"
-      (reference "C?") (unit 1) (value "1uF") (footprint "Capacitor_SMD:C_0603_1608Metric")
+      (reference "C14") (unit 1) (value "1uF") (footprint "Capacitor_SMD:C_0603_1608Metric")
     )
     (path "/c15641d3-3218-4ed3-b1f7-20e67018e0f9"
